File: pcbdesign/pcbdesign/pcbdesign.sch (KiCad schematic (older format))
At the start: 34 parts, among them J1 Conn_01x06_Male, J2 USB_B_Mini, J3 Conn_Coaxial, SW1 SW_Push, U1 CMWX1ZZABZ-078, U2 LM1117ADJ

Commit message: Add pull-up resistor to CS pin on SPI connector
Parts:
- added R?: 10K, symbol Device:R
- U1: symbol cmwx1zzabz-078:CMWX1ZZABZ-078 -> pcbdesign-rescue:CMWX1ZZABZ-078-cmwx1zzabz-078
- U2: symbol pcbdesign:LM1117ADJ -> pcbdesign-rescue:LM1117ADJ-pcbdesign
Connections:
- wire segments 149 -> 150
Changed lines of the file:
@@
 $EndDescr
 $Comp
-L cmwx1zzabz-078:CMWX1ZZABZ-078 U1
+L pcbdesign-rescue:CMWX1ZZABZ-078-cmwx1zzabz-078 U1
 U 1 1 5E390DC8
 P 7400 3550
@@
 $EndComp
 $Comp
-L pcbdesign:LM1117ADJ U2
+L pcbdesign-rescue:LM1117ADJ-pcbdesign U2
 U 1 1 5E4410B4
 P 3750 2450
@@
 CS
 Wire Wire Line
-	3150 6350 3500 6350
+	3150 6350 3400 6350
 Wire Wire Line
 	3150 6150 3500 6150
@@
 	1    0    0    -1
 $EndComp
+$Comp
+L Device:R R?
+U 1 1 5E3CC9AD
+P 3400 6500
+F 0 "R?" H 3470 6546 50  0000 L CNN
+F 1 "10K" H 3470 6455 50  0000 L CNN
+F 2 "" V 3330 6500 50  0001 C CNN
+F 3 "~" H 3400 6500 50  0001 C CNN
+	1    3400 6500
+	1    0    0    -1
+$EndComp
+Connection ~ 3400 6350
+Wire Wire Line
+	3400 6350 3500 6350
+$Comp
+L power:+3.3V #PWR?
+U 1 1 5E3CD027
+P 3400 6650
+F 0 "#PWR?" H 3400 6500 50  0001 C CNN
+F 1 "+3.3V" H 3415 6823 50  0000 C CNN
+F 2 "" H 3400 6650 50  0001 C CNN
+F 3 "" H 3400 6650 50  0001 C CNN
+	1    3400 6650
+	-1   0    0    1
+$EndComp
 $EndSCHEMATC
