File: pcbdesign/pcbdesign/pcbdesign.sch (KiCad schematic (older format))
At the start: 27 parts, among them J1 Conn_01x06_Male, J1 USB_B_Mini, SW1 SW_Push, SW2 SW_Push, U1 CMWX1ZZABZ-078, U2 LM1117ADJ

Commit message: Update pcbdesign
Parts:
- added Breathalizer1: Conn_01x04_Male, symbol Connector:Conn_01x04_Male
- added SSD1306-SPI: Conn_01x07_Male, symbol Connector:Conn_01x07_Male
Connections:
- net +3V3: now also Breathalizer1.2 (Pin_2), SSD1306-SPI.2 (Pin_2)
- net GND: now also Breathalizer1.1 (Pin_1), SSD1306-SPI.1 (Pin_1)
- new net CS: SSD1306-SPI.7 (Pin_7)
- new net D0: SSD1306-SPI.3 (Pin_3)
- new net D1: SSD1306-SPI.4 (Pin_4)
- new net DAT: Breathalizer1.4 (Pin_4)
- new net DC: SSD1306-SPI.6 (Pin_6)
- new net RES: SSD1306-SPI.5 (Pin_5)
- no-connect marks 40 -> 41
Changed lines of the file:
@@
 NoConn ~ 7500 2050
 NoConn ~ 7600 2050
+$Comp
+L Connector:Conn_01x04_Male Breathalizer1
+U 1 1 5E3B0FFE
+P 4650 6000
+F 0 "Breathalizer1" H 4758 6281 50  0000 C CNN
+F 1 "Conn_01x04_Male" H 4758 6190 50  0000 C CNN
+F 2 "" H 4650 6000 50  0001 C CNN
+F 3 "~" H 4650 6000 50  0001 C CNN
+	1    4650 6000
+	1    0    0    -1
+$EndComp
+$Comp
+L power:GND #PWR?
+U 1 1 5E3BA901
+P 5200 5800
+F 0 "#PWR?" H 5200 5550 50  0001 C CNN
+F 1 "GND" H 5205 5627 50  0000 C CNN
+F 2 "" H 5200 5800 50  0001 C CNN
+F 3 "" H 5200 5800 50  0001 C CNN
+	1    5200 5800
+	0    -1   -1   0
+$EndComp
+$Comp
+L power:+3.3V #PWR?
+U 1 1 5E3C65A3
+P 5200 6000
+F 0 "#PWR?" H 5200 5850 50  0001 C CNN
+F 1 "+3.3V" H 5215 6173 50  0000 C CNN
+F 2 "" H 5200 6000 50  0001 C CNN
+F 3 "" H 5200 6000 50  0001 C CNN
+	1    5200 6000
+	0    1    1    0
+$EndComp
+NoConn ~ 4850 6100
+Text Label 5200 6200 0    50   ~ 0
+DAT
+Wire Wire Line
+	4850 6200 5200 6200
+Wire Wire Line
+	4850 6000 5200 6000
+Wire Wire Line
+	4850 5900 5150 5900
+Wire Wire Line
+	5150 5900 5150 5800
+Wire Wire Line
+	5150 5800 5200 5800
+$Comp
+L power:GND #PWR?
+U 1 1 5E3EB6DF
+P 3700 5400
+F 0 "#PWR?" H 3700 5150 50  0001 C CNN
+F 1 "GND" H 3705 5227 50  0000 C CNN
+F 2 "" H 3700 5400 50  0001 C CNN
+F 3 "" H 3700 5400 50  0001 C CNN
+	1    3700 5400
+	-1   0    0    1
+$EndComp
+$Comp
+L power:+3.3V #PWR?
+U 1 1 5E3EBE04
+P 3950 5700
+F 0 "#PWR?" H 3950 5550 50  0001 C CNN
+F 1 "+3.3V" H 3965 5873 50  0000 C CNN
+F 2 "" H 3950 5700 50  0001 C CNN
+F 3 "" H 3950 5700 50  0001 C CNN
+	1    3950 5700
+	0    1    1    0
+$EndComp
+Text Label 3500 5950 0    50   ~ 0
+D0
+$Comp
+L Connector:Conn_01x07_Male SSD1306-SPI
+U 1 1 5E3E9C8E
+P 2950 6050
+F 0 "SSD1306-SPI" H 3058 6531 50  0000 C CNN
+F 1 "Conn_01x07_Male" H 3058 6440 50  0000 C CNN
+F 2 "" H 2950 6050 50  0001 C CNN
+F 3 "~" H 2950 6050 50  0001 C CNN
+	1    2950 6050
+	1    0    0    -1
+$EndComp
+Text Label 3500 6250 0    50   ~ 0
+DC
+Text Label 3500 6050 0    50   ~ 0
+D1
+Wire Wire Line
+	3150 5750 3700 5750
+Wire Wire Line
+	3700 5750 3700 5400
+Wire Wire Line
+	3150 5850 3800 5850
+Wire Wire Line
+	3800 5850 3800 5700
+Wire Wire Line
+	3800 5700 3950 5700
+Wire Wire Line
+	3150 5950 3500 5950
+Wire Wire Line
+	3150 6050 3500 6050
+Wire Wire Line
+	3150 6250 3500 6250
+Text Label 3500 6150 0    50   ~ 0
+RES
+Text Label 3500 6350 0    50   ~ 0
+CS
+Wire Wire Line
+	3150 6350 3500 6350
+Wire Wire Line
+	3150 6150 3500 6150
 $EndSCHEMATC

Commit message: Update pcbdesign
Parts:
- removed C7: 100n, symbol Device:C
- added C18, C19: 100n, Capacitor_SMD:C_0805_2012Metric, symbol Device:C
- added C20: 10n, Capacitor_SMD:C_0805_2012Metric, symbol Device:C
- added J3: Conn_Coaxial, symbol Connector:Conn_Coaxial
- added L1: L, symbol Device:L
- C1, C11, C12, C13, C15, C16, C2, C3, C4, C5, C6, C7, C8, C9: footprint (none) -> Capacitor_SMD:C_0805_2012Metric
- C10: renamed from C1; footprint (none) -> Capacitor_SMD:C_0805_2012Metric
- C14, C17: footprint (none) -> Capacitor_SMD:CP_Elec_5x5.3
- J1: footprint (none) -> Connector_PinHeader_2.54mm:PinHeader_1x06_P2.54mm_Vertical
- J2: renamed from J1; footprint (none) -> Connector_USB:USB_Mini-B_Wuerth_65100516121_Horizontal
- R1, R2, R3: footprint (none) -> Resistor_SMD:R_0805_2012Metric
- U2: footprint (none) -> Package_TO_SOT_SMD:SOT-223
- renumbered SSD1306-SPI to SSD1306-SPI1
Connections:
- net +3V3: now also C18.1
- net DAT: now also U1.24 (PA2/ADC2)
- net GND: now also C18.2, C19.2, C20.2, J3.2 (Ext)
- net at U1.26 (ANT): now also C19.1, L1.1
- new net: C20.1, J3.1 (In), L1.2
- no-connect marks 41 -> 39

Commit message: Update pcbdesign
Parts:
- removed L1: L, symbol Device:L
- removed R1: 10K, Resistor_SMD:R_0805_2012Metric, symbol Device:R
- removed SW2: SW_Push, symbol Switch:SW_Push
- added C21: 100p, Capacitor_SMD:C_0805_2012Metric, symbol Device:C
Connections:
- net +3V3: no longer Breathalizer1.2 (Pin_2)
- net +5V: now also Breathalizer1.2 (Pin_2)
- net at C19.1, U1.26 (ANT): now also C21.2
- net at C20.1, J3.1 (In): now also C21.1
- no-connect marks 39 -> 37
Other:
- moved on the sheet: Breathalizer1
Changed lines of the file:
@@
 Wire Wire Line
 	6350 4150 6350 4500
-$Comp
-L Switch:SW_Push SW1
-U 1 1 5E40E368
-P 5150 4550
-F 0 "SW1" V 5196 4502 50  0000 R CNN
-F 1 "SW_Push" V 5105 4502 50  0000 R CNN
-F 2 "" H 5150 4750 50  0001 C CNN
-F 3 "~" H 5150 4750 50  0001 C CNN
-	1    5150 4550
-	0    -1   -1   0
-$EndComp
 Wire Wire Line
 	6050 5000 6050 5200
@@
 	5150 4350 5150 4150
 NoConn ~ 9400 3100
-$Comp
-L Device:R R1
-U 1 1 5E428504
-P 6300 6350
-F 0 "R1" H 6370 6396 50  0000 L CNN
-F 1 "10K" H 6370 6305 50  0000 L CNN
-F 2 "Resistor_SMD:R_0805_2012Metric" V 6230 6350 50  0001 C CNN
-F 3 "~" H 6300 6350 50  0001 C CNN
-	1    6300 6350
-	1    0    0    -1
-$EndComp
-$Comp
-L Switch:SW_Push SW2
-U 1 1 5E42963C
-P 6300 5750
-F 0 "SW2" V 6346 5702 50  0000 R CNN
-F 1 "SW_Push" V 6255 5702 50  0000 R CNN
-F 2 "" H 6300 5950 50  0001 C CNN
-F 3 "~" H 6300 5950 50  0001 C CNN
-	1    6300 5750
-	0    -1   -1   0
-$EndComp
-$Comp
-L power:GND #PWR0108
-U 1 1 5E42EB00
-P 6300 6750
-F 0 "#PWR0108" H 6300 6500 50  0001 C CNN
-F 1 "GND" H 6305 6577 50  0000 C CNN
-F 2 "" H 6300 6750 50  0001 C CNN
-F 3 "" H 6300 6750 50  0001 C CNN
-	1    6300 6750
-	1    0    0    -1
-$EndComp
-Wire Wire Line
-	6300 6750 6300 6500
-Wire Wire Line
-	6300 6200 6300 5950
-Wire Wire Line
-	6300 5550 6300 4850
-Wire Wire Line
-	6300 4850 6500 4850
 $Comp
 L Connector:USB_B_Mini J2
@@
 	5850 1700 5850 1300
 NoConn ~ 6500 2650
-NoConn ~ 6500 2850
-NoConn ~ 6500 2950
-NoConn ~ 6500 3050
 NoConn ~ 6500 3150
 NoConn ~ 6500 3250
@@
 L Connector:Conn_01x04_Male Breathalizer1
 U 1 1 5E3B0FFE
-P 4650 6000
-F 0 "Breathalizer1" H 4758 6281 50  0000 C CNN
-F 1 "Conn_01x04_Male" H 4758 6190 50  0000 C CNN
-F 2 "" H 4650 6000 50  0001 C CNN
-F 3 "~" H 4650 6000 50  0001 C CNN
-	1    4650 6000
+P 5350 6000
+F 0 "Breathalizer1" H 5458 6281 50  0000 C CNN
+F 1 "Conn_01x04_Male" H 5458 6190 50  0000 C CNN
+F 2 "" H 5350 6000 50  0001 C CNN
+F 3 "~" H 5350 6000 50  0001 C CNN
+	1    5350 6000
 	1    0    0    -1
 $EndComp
@@
 L power:GND #PWR0118
 U 1 1 5E3BA901
-P 5200 5800
-F 0 "#PWR0118" H 5200 5550 50  0001 C CNN
-F 1 "GND" H 5205 5627 50  0000 C CNN
-F 2 "" H 5200 5800 50  0001 C CNN
-F 3 "" H 5200 5800 50  0001 C CNN
-	1    5200 5800
+P 5900 5800
+F 0 "#PWR0118" H 5900 5550 50  0001 C CNN
+F 1 "GND" H 5905 5627 50  0000 C CNN
+F 2 "" H 5900 5800 50  0001 C CNN
+F 3 "" H 5900 5800 50  0001 C CNN
+	1    5900 5800
 	0    -1   -1   0
 $EndComp
-$Comp
-L power:+3.3V #PWR0119
-U 1 1 5E3C65A3
-P 5200 6000
-F 0 "#PWR0119" H 5200 5850 50  0001 C CNN
-F 1 "+3.3V" H 5215 6173 50  0000 C CNN
-F 2 "" H 5200 6000 50  0001 C CNN
-F 3 "" H 5200 6000 50  0001 C CNN
-	1    5200 6000
-	0    1    1    0
-$EndComp
-NoConn ~ 4850 6100
-Text Label 5200 6200 0    50   ~ 0
+NoConn ~ 5550 6100
+Text Label 5900 6200 0    50   ~ 0
 DAT
 Wire Wire Line
-	4850 6200 5200 6200
-Wire Wire Line
-	4850 6000 5200 6000
-Wire Wire Line
-	4850 5900 5150 5900
-Wire Wire Line
-	5150 5900 5150 5800
-Wire Wire Line
-	5150 5800 5200 5800
+	5550 6200 5900 6200
+Wire Wire Line
+	5550 6000 5900 6000
+Wire Wire Line
+	5550 5900 5850 5900
+Wire Wire Line
+	5850 5900 5850 5800
+Wire Wire Line
+	5850 5800 5900 5800
 $Comp
 L power:GND #PWR0120
@@
 $EndComp
 $Comp
-L Device:L L1
-U 1 1 5E3C2D52
-P 9300 4850
-F 0 "L1" V 9490 4850 50  0000 C CNN
-F 1 "L" V 9399 4850 50  0000 C CNN
-F 2 "" H 9300 4850 50  0001 C CNN
-F 3 "~" H 9300 4850 50  0001 C CNN
-	1    9300 4850
-	0    -1   -1   0
-$EndComp
-$Comp
 L Device:C C19
 U 1 1 5E3C915C
@@
 Wire Wire Line
 	10350 4450 10350 4800
+NoConn ~ 6500 4850
+$Comp
+L Device:C C21
+U 1 1 5E415779
+P 9300 4850
+F 0 "C21" V 9048 4850 50  0000 C CNN
+F 1 "100p" V 9139 4850 50  0000 C CNN
+F 2 "Capacitor_SMD:C_0805_2012Metric" H 9338 4700 50  0001 C CNN
+F 3 "~" H 9300 4850 50  0001 C CNN
+	1    9300 4850
+	0    1    1    0
+$EndComp
+$Comp
+L Switch:SW_Push SW1
+U 1 1 5E40E368
+P 5150 4550
+F 0 "SW1" V 5196 4502 50  0000 R CNN
+F 1 "SW_Push" V 5105 4502 50  0000 R CNN
+F 2 "" H 5150 4750 50  0001 C CNN
+F 3 "~" H 5150 4750 50  0001 C CNN
+	1    5150 4550
+	0    -1   -1   0
+$EndComp
+$Comp
+L power:+5V #PWR?
+U 1 1 5E438F08
+P 5900 6000
+F 0 "#PWR?" H 5900 5850 50  0001 C CNN
+F 1 "+5V" H 5915 6173 50  0000 C CNN
+F 2 "" H 5900 6000 50  0001 C CNN
+F 3 "" H 5900 6000 50  0001 C CNN
+	1    5900 6000
+	0    1    1    0
+$EndComp
 $EndSCHEMATC

Commit message: Update pcbdesign
Parts:
- added BZ1: Buzzer, symbol Device:Buzzer
- added R4: 680, Resistor_SMD:R_0805_2012Metric, symbol Device:R
- added R5: 1200, Resistor_SMD:R_0805_2012Metric, symbol Device:R
- Breathalizer1: footprint (none) -> Connector_PinHeader_2.54mm:PinHeader_1x04_P2.54mm_Vertical
- R2: value 500 -> 680
- SSD1306-SPI1: footprint (none) -> Connector_PinHeader_2.54mm:PinHeader_1x07_P2.54mm_Vertical
- SW1: footprint (none) -> Button_Switch_SMD:SW_Push_1P1T_NO_6x6mm_H9.5mm
Connections:
- net CS: now also U1.17 (PB12/SPI2_NSS)
- net D0: now also U1.16 (PB13/SPI2_SCK)
- net D1: now also U1.14 (PB15/SPI2_MOSI)
- net DAT: now also R4.2, R5.1; no longer Breathalizer1.4 (Pin_4)
- net DC: now also U1.35 (PB8/I2C1_SCL)
- net GND: now also R5.2
- net RES: now also U1.36 (PB9/I2C1_SDA)
- new net: Breathalizer1.4 (Pin_4), R4.1
- no-connect marks 37 -> 34
Changed lines of the file:
@@
 P 4500 2150
 F 0 "R2" H 4570 2196 50  0000 L CNN
-F 1 "500" H 4570 2105 50  0000 L CNN
+F 1 "680" H 4570 2105 50  0000 L CNN
 F 2 "Resistor_SMD:R_0805_2012Metric" V 4430 2150 50  0001 C CNN
 F 3 "~" H 4500 2150 50  0001 C CNN
@@
 NoConn ~ 8300 3850
 NoConn ~ 8300 3750
-NoConn ~ 8300 3550
 NoConn ~ 8300 3450
-NoConn ~ 8300 3350
-NoConn ~ 8300 3250
-NoConn ~ 8300 3150
-NoConn ~ 8300 3050
 NoConn ~ 8300 2950
 NoConn ~ 8300 2850
@@
 F 0 "Breathalizer1" H 5458 6281 50  0000 C CNN
 F 1 "Conn_01x04_Male" H 5458 6190 50  0000 C CNN
-F 2 "" H 5350 6000 50  0001 C CNN
+F 2 "Connector_PinHeader_2.54mm:PinHeader_1x04_P2.54mm_Vertical" H 5350 6000 50  0001 C CNN
 F 3 "~" H 5350 6000 50  0001 C CNN
 	1    5350 6000
@@
 $EndComp
 NoConn ~ 5550 6100
-Text Label 5900 6200 0    50   ~ 0
+Text Label 7000 6200 0    50   ~ 0
 DAT
-Wire Wire Line
-	5550 6200 5900 6200
 Wire Wire Line
 	5550 6000 5900 6000
@@
 F 0 "SSD1306-SPI1" H 3058 6531 50  0000 C CNN
 F 1 "Conn_01x07_Male" H 3058 6440 50  0000 C CNN
-F 2 "" H 2950 6050 50  0001 C CNN
+F 2 "Connector_PinHeader_2.54mm:PinHeader_1x07_P2.54mm_Vertical" H 2950 6050 50  0001 C CNN
 F 3 "~" H 2950 6050 50  0001 C CNN
 	1    2950 6050
@@
 F 0 "SW1" V 5196 4502 50  0000 R CNN
 F 1 "SW_Push" V 5105 4502 50  0000 R CNN
-F 2 "" H 5150 4750 50  0001 C CNN
+F 2 "Button_Switch_SMD:SW_Push_1P1T_NO_6x6mm_H9.5mm" H 5150 4750 50  0001 C CNN
 F 3 "~" H 5150 4750 50  0001 C CNN
 	1    5150 4550
@@
 $EndComp
 $Comp
-L power:+5V #PWR?
+L power:+5V #PWR0108
 U 1 1 5E438F08
 P 5900 6000
-F 0 "#PWR?" H 5900 5850 50  0001 C CNN
+F 0 "#PWR0108" H 5900 5850 50  0001 C CNN
 F 1 "+5V" H 5915 6173 50  0000 C CNN
 F 2 "" H 5900 6000 50  0001 C CNN
@@
 	0    1    1    0
 $EndComp
+$Comp
+L Device:R R4
+U 1 1 5E459340
+P 6100 6400
+F 0 "R4" H 6170 6446 50  0000 L CNN
+F 1 "680" H 6170 6355 50  0000 L CNN
+F 2 "Resistor_SMD:R_0805_2012Metric" V 6030 6400 50  0001 C CNN
+F 3 "~" H 6100 6400 50  0001 C CNN
+	1    6100 6400
+	1    0    0    -1
+$EndComp
+$Comp
+L Device:R R5
+U 1 1 5E459B97
+P 6100 6850
+F 0 "R5" H 6170 6896 50  0000 L CNN
+F 1 "1200" H 6170 6805 50  0000 L CNN
+F 2 "Resistor_SMD:R_0805_2012Metric" V 6030 6850 50  0001 C CNN
+F 3 "~" H 6100 6850 50  0001 C CNN
+	1    6100 6850
+	1    0    0    -1
+$EndComp
+Wire Wire Line
+	5550 6200 6100 6200
+Wire Wire Line
+	6100 6200 6100 6250
+Wire Wire Line
+	6100 6550 6100 6600
+$Comp
+L power:GND #PWR0119
+U 1 1 5E4E6167
+P 6100 7200
+F 0 "#PWR0119" H 6100 6950 50  0001 C CNN
+F 1 "GND" H 6105 7027 50  0000 C CNN
+F 2 "" H 6100 7200 50  0001 C CNN
+F 3 "" H 6100 7200 50  0001 C CNN
+	1    6100 7200
+	1    0    0    -1
+$EndComp
+Wire Wire Line
+	6100 7200 6100 7000
+Wire Wire Line
+	6100 6600 6500 6600
+Wire Wire Line
+	6500 6600 6500 6200
+Wire Wire Line
+	6500 6200 7000 6200
+Connection ~ 6100 6600
+Wire Wire Line
+	6100 6600 6100 6700
+Text Label 8700 3250 0    50   ~ 0
+CS
+Wire Wire Line
+	8300 3250 8700 3250
+Text Label 8700 3350 0    50   ~ 0
+D0
+Wire Wire Line
+	8300 3350 8700 3350
+Text Label 8700 3550 0    50   ~ 0
+D1
+Wire Wire Line
+	8300 3550 8700 3550
+NoConn ~ 6500 3050
+NoConn ~ 6500 2950
+Text Label 8700 3050 0    50   ~ 0
+DC
+Text Label 8700 3150 0    50   ~ 0
+RES
+Wire Wire Line
+	8300 3150 8700 3150
+Wire Wire Line
+	8300 3050 8700 3050
+$Comp
+L Device:Buzzer BZ1
+U 1 1 5E5528D6
+P 5350 3050
+F 0 "BZ1" H 5355 3340 50  0000 C CNN
+F 1 "Buzzer" H 5355 3249 50  0000 C CNN
+F 2 "" V 5325 3150 50  0001 C CNN
+F 3 "~" V 5325 3150 50  0001 C CNN
+	1    5350 3050
+	-1   0    0    -1
+$EndComp
+$Comp
+L power:GND #PWR0125
+U 1 1 5E55FF58
+P 5800 3200
+F 0 "#PWR0125" H 5800 2950 50  0001 C CNN
+F 1 "GND" H 5805 3027 50  0000 C CNN
+F 2 "" H 5800 3200 50  0001 C CNN
+F 3 "" H 5800 3200 50  0001 C CNN
+	1    5800 3200
+	1    0    0    -1
+$EndComp
 $EndSCHEMATC

Commit message: Update pcbdesign
Parts:
- SW1: footprint Button_Switch_SMD:SW_Push_1P1T_NO_6x6mm_H9.5mm -> (none)
Connections:
- net GND: now also SW1.2; no longer SW1.1
- net NRST: now also SW1.1; no longer SW1.2
Changed lines of the file:
@@
 	6500 3950 6050 3950
 Wire Wire Line
-	6050 3950 6050 4150
-Wire Wire Line
-	5150 4150 6050 4150
+	6050 3950 6050 4050
 Connection ~ 6050 4150
 Wire Wire Line
@@
 Wire Wire Line
 	6350 4150 6350 4500
-Wire Wire Line
-	6050 5000 6050 5200
-Wire Wire Line
-	5150 4750 5150 5000
-Wire Wire Line
-	5150 5000 6050 5000
-Wire Wire Line
-	6050 5000 6050 4700
-Connection ~ 6050 5000
-Wire Wire Line
-	5150 4350 5150 4150
 NoConn ~ 9400 3100
 $Comp
@@
 $EndComp
 $Comp
-L Switch:SW_Push SW1
-U 1 1 5E40E368
-P 5150 4550
-F 0 "SW1" V 5196 4502 50  0000 R CNN
-F 1 "SW_Push" V 5105 4502 50  0000 R CNN
-F 2 "Button_Switch_SMD:SW_Push_1P1T_NO_6x6mm_H9.5mm" H 5150 4750 50  0001 C CNN
-F 3 "~" H 5150 4750 50  0001 C CNN
-	1    5150 4550
-	0    -1   -1   0
-$EndComp
-$Comp
 L power:+5V #PWR0108
 U 1 1 5E438F08
@@
 	1    0    0    -1
 $EndComp
+Wire Wire Line
+	6050 4700 6050 5000
+$Comp
+L Switch:SW_Push SW1
+U 1 1 5E63CCBC
+P 5150 4550
+F 0 "SW1" V 5104 4698 50  0000 L CNN
+F 1 "SW_Push" V 5195 4698 50  0000 L CNN
+F 2 "" H 5150 4750 50  0001 C CNN
+F 3 "~" H 5150 4750 50  0001 C CNN
+	1    5150 4550
+	0    1    1    0
+$EndComp
+Wire Wire Line
+	5150 4350 5150 4050
+Wire Wire Line
+	5150 4050 6050 4050
+Connection ~ 6050 4050
+Wire Wire Line
+	6050 4050 6050 4150
+Wire Wire Line
+	5150 4750 5150 5000
+Wire Wire Line
+	5150 5000 6050 5000
+Connection ~ 6050 5000
+Wire Wire Line
+	6050 5000 6050 5200
 $EndSCHEMATC
