File: pcbdesign/pcbdesign/_autosave-pcbdesign.sch (KiCad schematic (older format))
At the start: 35 parts, among them J1 Conn_01x06_Male, J2 USB_B_Mini, J3 Conn_Coaxial, SW1 SW_Push, U1 CMWX1ZZABZ-078, U2 LM1117ADJ

Commit message: Place components on PCB
Parts:
- removed C18: 4.7u, Capacitor_SMD:C_0805_2012Metric, symbol Device:C
- removed C2, C3, C4, C5, C6: 100n, Capacitor_SMD:C_0805_2012Metric, symbol Device:C
Changed lines of the file:
@@
 	1    0    0    -1
 $EndComp
-$Comp
-L Device:C C2
-U 1 1 5E392739
-P 1950 4200
-F 0 "C2" H 2065 4246 50  0000 L CNN
-F 1 "100n" H 2065 4155 50  0000 L CNN
-F 2 "Capacitor_SMD:C_0805_2012Metric" H 1988 4050 50  0001 C CNN
-F 3 "~" H 1950 4200 50  0001 C CNN
-	1    1950 4200
-	1    0    0    -1
-$EndComp
-$Comp
-L Device:C C5
-U 1 1 5E392DF0
-P 3300 4200
-F 0 "C5" H 3415 4246 50  0000 L CNN
-F 1 "100n" H 3415 4155 50  0000 L CNN
-F 2 "Capacitor_SMD:C_0805_2012Metric" H 3338 4050 50  0001 C CNN
-F 3 "~" H 3300 4200 50  0001 C CNN
-	1    3300 4200
-	1    0    0    -1
-$EndComp
-$Comp
-L Device:C C6
-U 1 1 5E3930A1
-P 3750 4200
-F 0 "C6" H 3865 4246 50  0000 L CNN
-F 1 "100n" H 3865 4155 50  0000 L CNN
-F 2 "Capacitor_SMD:C_0805_2012Metric" H 3788 4050 50  0001 C CNN
-F 3 "~" H 3750 4200 50  0001 C CNN
-	1    3750 4200
-	1    0    0    -1
-$EndComp
-$Comp
-L Device:C C3
-U 1 1 5E393437
-P 2400 4200
-F 0 "C3" H 2515 4246 50  0000 L CNN
-F 1 "100n" H 2515 4155 50  0000 L CNN
-F 2 "Capacitor_SMD:C_0805_2012Metric" H 2438 4050 50  0001 C CNN
-F 3 "~" H 2400 4200 50  0001 C CNN
-	1    2400 4200
-	1    0    0    -1
-$EndComp
-$Comp
-L Device:C C4
-U 1 1 5E3938B4
-P 2850 4200
-F 0 "C4" H 2965 4246 50  0000 L CNN
-F 1 "100n" H 2965 4155 50  0000 L CNN
-F 2 "Capacitor_SMD:C_0805_2012Metric" H 2888 4050 50  0001 C CNN
-F 3 "~" H 2850 4200 50  0001 C CNN
-	1    2850 4200
-	1    0    0    -1
-$EndComp
-$Comp
-L power:GND #PWR0101
-U 1 1 5E399258
-P 3050 4850
-F 0 "#PWR0101" H 3050 4600 50  0001 C CNN
-F 1 "GND" H 3055 4677 50  0000 C CNN
-F 2 "" H 3050 4850 50  0001 C CNN
-F 3 "" H 3050 4850 50  0001 C CNN
-	1    3050 4850
-	1    0    0    -1
-$EndComp
-Wire Wire Line
-	3050 4650 3050 4850
-Connection ~ 3050 4650
-$Comp
-L power:+3.3V #PWR0102
-U 1 1 5E39BDD6
-P 3050 3650
-F 0 "#PWR0102" H 3050 3500 50  0001 C CNN
-F 1 "+3.3V" H 3065 3823 50  0000 C CNN
-F 2 "" H 3050 3650 50  0001 C CNN
-F 3 "" H 3050 3650 50  0001 C CNN
-	1    3050 3650
-	1    0    0    -1
-$EndComp
-Wire Wire Line
-	3050 3800 3050 3650
-Connection ~ 3050 3800
-Wire Wire Line
-	3050 4650 3300 4650
-Wire Wire Line
-	1950 4650 2400 4650
-Wire Wire Line
-	1950 3800 2400 3800
-Wire Wire Line
-	3050 3800 3300 3800
-Wire Wire Line
-	4200 4050 4200 3800
-Wire Wire Line
-	3750 4050 3750 3800
-Connection ~ 3750 3800
-Wire Wire Line
-	3750 3800 4200 3800
-Wire Wire Line
-	3300 4050 3300 3800
-Connection ~ 3300 3800
-Wire Wire Line
-	3300 3800 3750 3800
-Wire Wire Line
-	3300 4350 3300 4650
-Connection ~ 3300 4650
-Wire Wire Line
-	3300 4650 3750 4650
-Wire Wire Line
-	3750 4350 3750 4650
-Connection ~ 3750 4650
-Wire Wire Line
-	3750 4650 4200 4650
-Wire Wire Line
-	4200 4350 4200 4650
-Wire Wire Line
-	2850 4350 2850 4650
-Connection ~ 2850 4650
-Wire Wire Line
-	2850 4650 3050 4650
-Wire Wire Line
-	2850 4050 2850 3800
-Connection ~ 2850 3800
-Wire Wire Line
-	2850 3800 3050 3800
-Wire Wire Line
-	2400 4050 2400 3800
-Connection ~ 2400 3800
-Wire Wire Line
-	2400 3800 2850 3800
-Wire Wire Line
-	1950 4050 1950 3800
-Wire Wire Line
-	1950 4350 1950 4650
-Wire Wire Line
-	2400 4350 2400 4650
-Connection ~ 2400 4650
-Wire Wire Line
-	2400 4650 2850 4650
 Text Label 5750 3800 0    50   ~ 0
 SWCLK
@@
 NoConn ~ 9400 3100
 $Comp
-L Connector:USB_B_Mini J2
-U 1 1 5E434262
-P 1150 1850
-F 0 "J2" H 1207 2317 50  0000 C CNN
-F 1 "USB_B_Mini" H 1207 2226 50  0000 C CNN
-F 2 "Connector_USB:USB_Mini-B_Wuerth_65100516121_Horizontal" H 1300 1800 50  0001 C CNN
-F 3 "~" H 1300 1800 50  0001 C CNN
-	1    1150 1850
-	1    0    0    -1
-$EndComp
-$Comp
 L pcbdesign-rescue:LM1117ADJ-pcbdesign U2
 U 1 1 5E4410B4
@@
 $EndComp
 Wire Wire Line
-	1050 2250 1050 2450
-Wire Wire Line
 	1050 2450 1100 2450
-Wire Wire Line
-	1150 2450 1150 2250
-Wire Wire Line
-	1100 2450 1100 2600
 Connection ~ 1100 2450
 Wire Wire Line
 	1100 2450 1150 2450
-NoConn ~ 1450 1850
-NoConn ~ 1450 1950
-NoConn ~ 1450 2050
-$Comp
-L Device:C C13
-U 1 1 5E44EB5B
-P 1800 1800
-F 0 "C13" H 1915 1846 50  0000 L CNN
-F 1 "100n" H 1915 1755 50  0000 L CNN
-F 2 "Capacitor_SMD:C_0805_2012Metric" H 1838 1650 50  0001 C CNN
-F 3 "~" H 1800 1800 50  0001 C CNN
-	1    1800 1800
-	1    0    0    -1
-$EndComp
-$Comp
-L Device:C C15
-U 1 1 5E44F841
-P 2700 1800
-F 0 "C15" H 2815 1846 50  0000 L CNN
-F 1 "100n" H 2815 1755 50  0000 L CNN
-F 2 "Capacitor_SMD:C_0805_2012Metric" H 2738 1650 50  0001 C CNN
-F 3 "~" H 2700 1800 50  0001 C CNN
-	1    2700 1800
-	1    0    0    -1
-$EndComp
-$Comp
-L power:GND #PWR0110
-U 1 1 5E45012F
-P 1800 2150
-F 0 "#PWR0110" H 1800 1900 50  0001 C CNN
-F 1 "GND" H 1805 1977 50  0000 C CNN
-F 2 "" H 1800 2150 50  0001 C CNN
-F 3 "" H 1800 2150 50  0001 C CNN
-	1    1800 2150
-	1    0    0    -1
-$EndComp
-$Comp
-L power:GND #PWR0111
-U 1 1 5E4510F7
-P 2250 2150
-F 0 "#PWR0111" H 2250 1900 50  0001 C CNN
-F 1 "GND" H 2255 1977 50  0000 C CNN
-F 2 "" H 2250 2150 50  0001 C CNN
-F 3 "" H 2250 2150 50  0001 C CNN
-	1    2250 2150
-	1    0    0    -1
-$EndComp
-$Comp
-L power:GND #PWR0112
-U 1 1 5E452DFE
-P 2700 2150
-F 0 "#PWR0112" H 2700 1900 50  0001 C CNN
-F 1 "GND" H 2705 1977 50  0000 C CNN
-F 2 "" H 2700 2150 50  0001 C CNN
-F 3 "" H 2700 2150 50  0001 C CNN
-	1    2700 2150
-	1    0    0    -1
-$EndComp
 $Comp
 L power:GND #PWR0113
@@
 	1    0    0    -1
 $EndComp
-$Comp
-L Device:CP C14
-U 1 1 5E45AA6F
-P 2250 1800
-F 0 "C14" H 2368 1846 50  0000 L CNN
-F 1 "10u" H 2368 1755 50  0000 L CNN
-F 2 "Capacitor_SMD:CP_Elec_5x5.3" H 2288 1650 50  0001 C CNN
-F 3 "~" H 2250 1800 50  0001 C CNN
-	1    2250 1800
-	1    0    0    -1
-$EndComp
-Wire Wire Line
-	1450 1650 1600 1650
-Connection ~ 1800 1650
-Wire Wire Line
-	1800 1650 2250 1650
-Connection ~ 2250 1650
-Wire Wire Line
-	2250 1650 2700 1650
-Wire Wire Line
-	1800 2150 1800 1950
-Wire Wire Line
-	2250 2150 2250 1950
-Wire Wire Line
-	2700 2150 2700 1950
-Wire Wire Line
-	2700 1650 3150 1650
-Wire Wire Line
-	3150 1650 3150 2050
-Wire Wire Line
-	3150 2050 3400 2050
-Connection ~ 2700 1650
-$Comp
-L power:+5V #PWR0115
-U 1 1 5E484268
-P 1600 1450
-F 0 "#PWR0115" H 1600 1300 50  0001 C CNN
-F 1 "+5V" H 1615 1623 50  0000 C CNN
-F 2 "" H 1600 1450 50  0001 C CNN
-F 3 "" H 1600 1450 50  0001 C CNN
-	1    1600 1450
-	1    0    0    -1
-$EndComp
-Wire Wire Line
-	1600 1650 1600 1450
-Connection ~ 1600 1650
-Wire Wire Line
-	1600 1650 1800 1650
 $Comp
 L Device:R R2
@@
 $EndComp
 $Comp
-L Device:C C18
-U 1 1 5E500834
-P 4200 4200
-F 0 "C18" H 4315 4246 50  0000 L CNN
-F 1 "4.7u" H 4315 4155 50  0000 L CNN
-F 2 "Capacitor_SMD:C_0805_2012Metric" H 4238 4050 50  0001 C CNN
-F 3 "~" H 4200 4200 50  0001 C CNN
-	1    4200 4200
-	1    0    0    -1
-$EndComp
-$Comp
 L power:GND #PWR0122
 U 1 1 5E3B87DE
@@
 	0    -1   -1   0
 $EndComp
+Wire Wire Line
+	1100 2450 1100 2600
+Wire Wire Line
+	1600 1650 1800 1650
+Connection ~ 1600 1650
+Wire Wire Line
+	1600 1650 1600 1450
+$Comp
+L power:+5V #PWR0115
+U 1 1 5E484268
+P 1600 1450
+F 0 "#PWR0115" H 1600 1300 50  0001 C CNN
+F 1 "+5V" H 1615 1623 50  0000 C CNN
+F 2 "" H 1600 1450 50  0001 C CNN
+F 3 "" H 1600 1450 50  0001 C CNN
+	1    1600 1450
+	1    0    0    -1
+$EndComp
+Connection ~ 2700 1650
+Wire Wire Line
+	3150 2050 3400 2050
+Wire Wire Line
+	3150 1650 3150 2050
+Wire Wire Line
+	2700 1650 3150 1650
+Wire Wire Line
+	2700 2150 2700 1950
+Wire Wire Line
+	2250 2150 2250 1950
+Wire Wire Line
+	1800 2150 1800 1950
+Wire Wire Line
+	2250 1650 2700 1650
+Connection ~ 2250 1650
+Wire Wire Line
+	1800 1650 2250 1650
+Connection ~ 1800 1650
+Wire Wire Line
+	1450 1650 1600 1650
+$Comp
+L Device:CP C14
+U 1 1 5E45AA6F
+P 2250 1800
+F 0 "C14" H 2368 1846 50  0000 L CNN
+F 1 "10u" H 2368 1755 50  0000 L CNN
+F 2 "Capacitor_SMD:CP_Elec_5x5.3" H 2288 1650 50  0001 C CNN
+F 3 "~" H 2250 1800 50  0001 C CNN
+	1    2250 1800
+	1    0    0    -1
+$EndComp
+$Comp
+L power:GND #PWR0112
+U 1 1 5E452DFE
+P 2700 2150
+F 0 "#PWR0112" H 2700 1900 50  0001 C CNN
+F 1 "GND" H 2705 1977 50  0000 C CNN
+F 2 "" H 2700 2150 50  0001 C CNN
+F 3 "" H 2700 2150 50  0001 C CNN
+	1    2700 2150
+	1    0    0    -1
+$EndComp
+$Comp
+L power:GND #PWR0111
+U 1 1 5E4510F7
+P 2250 2150
+F 0 "#PWR0111" H 2250 1900 50  0001 C CNN
+F 1 "GND" H 2255 1977 50  0000 C CNN
+F 2 "" H 2250 2150 50  0001 C CNN
+F 3 "" H 2250 2150 50  0001 C CNN
+	1    2250 2150
+	1    0    0    -1
+$EndComp
+$Comp
+L power:GND #PWR0110
+U 1 1 5E45012F
+P 1800 2150
+F 0 "#PWR0110" H 1800 1900 50  0001 C CNN
+F 1 "GND" H 1805 1977 50  0000 C CNN
+F 2 "" H 1800 2150 50  0001 C CNN
+F 3 "" H 1800 2150 50  0001 C CNN
+	1    1800 2150
+	1    0    0    -1
+$EndComp
+$Comp
+L Device:C C15
+U 1 1 5E44F841
+P 2700 1800
+F 0 "C15" H 2815 1846 50  0000 L CNN
+F 1 "100n" H 2815 1755 50  0000 L CNN
+F 2 "Capacitor_SMD:C_0805_2012Metric" H 2738 1650 50  0001 C CNN
+F 3 "~" H 2700 1800 50  0001 C CNN
+	1    2700 1800
+	1    0    0    -1
+$EndComp
+$Comp
+L Device:C C13
+U 1 1 5E44EB5B
+P 1800 1800
+F 0 "C13" H 1915 1846 50  0000 L CNN
+F 1 "100n" H 1915 1755 50  0000 L CNN
+F 2 "Capacitor_SMD:C_0805_2012Metric" H 1838 1650 50  0001 C CNN
+F 3 "~" H 1800 1800 50  0001 C CNN
+	1    1800 1800
+	1    0    0    -1
+$EndComp
+NoConn ~ 1450 2050
+NoConn ~ 1450 1950
+NoConn ~ 1450 1850
+Wire Wire Line
+	1150 2450 1150 2250
+Wire Wire Line
+	1050 2250 1050 2450
+$Comp
+L Connector:USB_B_Mini J2
+U 1 1 5E434262
+P 1150 1850
+F 0 "J2" H 1207 2317 50  0000 C CNN
+F 1 "USB_B_Mini" H 1207 2226 50  0000 C CNN
+F 2 "Connector_USB:USB_Mini-B_Wuerth_65100516121_Horizontal" H 1300 1800 50  0001 C CNN
+F 3 "~" H 1300 1800 50  0001 C CNN
+	1    1150 1850
+	1    0    0    -1
+$EndComp
 $EndSCHEMATC
